File: tool/kicad/shape2/shape.kicad_pcb (KiCad board)
At the start: 2 copper layers, 30 x 20 mm, 22 parts, among them K1 CONN_3, P31 CONN_7, U1 MCP6022, U2 MCP6022

Commit message: layout
Parts:
- removed C10: 1nF, pretty:0603_S
- removed C9: 1uF, pretty:0603_S
- removed D2, D3: D, pretty:0805_LED
- removed K1: CONN_3, pretty:PIN_1X3
- added C11: 1pF?, pretty:0603_S, F.Cu at (76.3, 106.6)
- added C12: 1pF?, pretty:0603_S, F.Cu at (76.3, 98.7)
- added R10: 100k, pretty:0603_S_R, F.Cu at (76.3, 103.4)
- added R11: 100k, pretty:0603_S_R, F.Cu at (76.3, 95.5)
- added R6: 100k, pretty:0603_S_R, F.Cu at (73.8, 99.6)
- added R7: 100k, pretty:0603_S_R, F.Cu at (73.8, 97.4)
- added R8: 33k, pretty:0603_S_R, F.Cu at (82.2, 101.0)
- added R9: 33k, pretty:0603_S_R, F.Cu at (82.1, 92.9)
- added RV1: 10k, pretty:SMT_trimmer_Panasonic_EVM3Y, F.Cu at (71.2, 106.2)
- C2: value 0.1uF -> 1uF
- C4: value 0.1uF -> 1pF?
- C6: value 1uF -> 1pF?
- R2: value R -> 1k
- R3: value R -> 1.5k
- R4, R5: value R -> 33k
- moved C1 19.5 mm to (89.5, 93.9), turned to 270 degrees
- moved R3 17.7 mm to (74.3, 107.8)
- moved R4 17.2 mm to (70.5, 99.6), turned to 0 degrees
- moved C2 17.2 mm to (87.8, 93.9), turned to 270 degrees
- moved R5 16.5 mm to (70.5, 97.4), turned to 0 degrees
- moved R2 14.8 mm to (74.3, 104.6)
- moved C4 12.5 mm to (87.8, 105.5)
- moved C6 6.13 mm to (87.9, 97.6), turned to 90 degrees
- moved C3 3.51 mm to (87.8, 101.7), turned to 270 degrees
- moved C5 2.60 mm to (89.5, 101.7), turned to 270 degrees
- moved C8 1.27 mm to (71.6, 102.1)
- moved C7 1.14 mm to (69.8, 102.1)
- moved U1 1.00 mm to (82.0, 104.5)
- moved U2 1.00 mm to (82.0, 96.5)
Connections:
- C1 pad 1: /MO -> GND
- C1 pad 2: /MOA -> +5V
- C2 pad 1: /RO -> GND
- C2 pad 2: /ROA -> +5V
- C4 pad 2: +5V -> /MO_SAMPLE
- C6 pad 2: +5V -> /RO_SAMPLE
- R2 pad 1: Net-(R2-Pad1) -> +5V
- R2 pad 2: GND -> /VSUB
- R3 pad 1: Net-(R3-Pad1) -> /VSUB
- R4 pad 1: /MO_SAMPLE -> /MO
- R4 pad 2: Net-(R2-Pad1) -> /MOA
- R5 pad 1: /RO_SAMPLE -> /RO
- R5 pad 2: Net-(R3-Pad1) -> /ROA
- U1 pad 1: /MOO -> Net-(R10-Pad1)
- U1 pad 2: /MOA -> /MOO
- U1 pad 3: GND -> /MOA
- U1 pad 6: Net-(R2-Pad1) -> /MO_SAMPLE
- U2 pad 1: /ROO -> Net-(R11-Pad1)
- U2 pad 2: /ROA -> /ROO
- U2 pad 3: GND -> /ROA
- U2 pad 6: Net-(R3-Pad1) -> /RO_SAMPLE
Routing:
- net /VSUB: track 0.00 -> 47.2 mm, vias 0 -> 3
- net +3.3V: track 39.3 -> 0.00 mm
- net GND: track 0.00 -> 15.3 mm, vias 0 -> 12
- net +5V: track 71.8 -> 64.2 mm
- net /MO_SAMPLE: track 23.3 -> 28.3 mm, vias 1 -> 2
- net Net-(R2-Pad1): track 4.81 -> 0.00 mm
- net Net-(R3-Pad1): track 4.77 -> 0.00 mm
- net /MOO: track 12.1 -> 16.8 mm
- net /ROO: track 12.1 -> 16.8 mm
- net /MOA: track 8.93 -> 12.5 mm, vias 0 -> 2
- net /ROA: track 6.77 -> 10.4 mm, vias 0 -> 2
- net Net-(R11-Pad1): track 0.00 -> 2.32 mm
- net Net-(R10-Pad1): track 0.00 -> 2.32 mm
- net /RO_SAMPLE: track 21.1 -> 23.3 mm, vias 1 -> 2
Other:
- board text added: "v2"
- board text removed: "v1"
