File: tool/kicad/shape2/shape.sch (KiCad schematic (older format))
At the start: 22 parts, among them K1 CONN_3, P31 CONN_7, U1 MCP6022, U2 MCP6022

Commit message: layout
Parts:
- removed C10: 1nF, symbol C
- removed C9: 1uF, symbol C
- removed D2, D3: D, symbol D
- removed K1: CONN_3, symbol CONN_3
- added C11, C12: 1pF?, symbol C
- added R10, R11, R6, R7: 100k, symbol R
- added R8, R9: 33k, symbol R
- added RV1: 10k, symbol POT
- C2: value 0.1uF -> 1uF
- C4: value 0.1uF -> 1pF?
- C6: value 1uF -> 1pF?
- R2: value R -> 1k
- R3: value R -> 1.5k
- R4, R5: value R -> 33k
Connections:
- net labels added: VSUB
- wire segments 97 -> 90
