File: tool/kicad/shape/shape.sch (KiCad schematic (older format))
At the start: 29 parts, among them K1 CONN_3, P1 CONN_7, U1 MCP6022

Commit message: tune shape board
Parts:
- R1, R2: value 2.2k -> 0/2.2k
- R10: value 1.5k -> 1.1k
- R3, R4, R7, R8: value 33k -> 56.2k
- R9: value 1k -> 1.21k
Changed lines of the file:
@@
 P 2850 1250
 F 0 "R9" H 2850 1300 40  0000 C CNN
-F 1 "1k" H 2850 1200 40  0000 C CNN
+F 1 "1.21k" H 2850 1200 40  0000 C CNN
 F 2 "" H 2850 1250 60  0000 C CNN
 F 3 "" H 2850 1250 60  0000 C CNN
@@
 P 2850 1450
 F 0 "R10" H 2850 1500 40  0000 C CNN
-F 1 "1.5k" H 2850 1400 40  0000 C CNN
+F 1 "1.1k" H 2850 1400 40  0000 C CNN
 F 2 "" H 2850 1450 60  0000 C CNN
 F 3 "" H 2850 1450 60  0000 C CNN
@@
 P 2400 2650
 F 0 "R7" H 2400 2700 40  0000 C CNN
-F 1 "33k" H 2400 2600 40  0000 C CNN
+F 1 "56.2k" H 2400 2600 40  0000 C CNN
 F 2 "" H 2400 2650 60  0000 C CNN
 F 3 "" H 2400 2650 60  0000 C CNN
@@
 P 1850 2750
 F 0 "R3" H 1850 2800 40  0000 C CNN
-F 1 "33k" H 1850 2700 40  0000 C CNN
+F 1 "56.2k" H 1850 2700 40  0000 C CNN
 F 2 "" H 1850 2750 60  0000 C CNN
 F 3 "" H 1850 2750 60  0000 C CNN
@@
 P 1500 2750
 F 0 "R1" H 1500 2800 40  0000 C CNN
-F 1 "2.2k" H 1500 2700 40  0000 C CNN
+F 1 "0/2.2k" H 1500 2700 40  0000 C CNN
 F 2 "" H 1500 2750 60  0000 C CNN
 F 3 "" H 1500 2750 60  0000 C CNN
@@
 P 2400 2950
 F 0 "R8" H 2400 3000 40  0000 C CNN
-F 1 "33k" H 2400 2900 40  0000 C CNN
+F 1 "56.2k" H 2400 2900 40  0000 C CNN
 F 2 "" H 2400 2950 60  0000 C CNN
 F 3 "" H 2400 2950 60  0000 C CNN
@@
 P 1850 3250
 F 0 "R4" H 1850 3300 40  0000 C CNN
-F 1 "33k" H 1850 3200 40  0000 C CNN
+F 1 "56.2k" H 1850 3200 40  0000 C CNN
 F 2 "" H 1850 3250 60  0000 C CNN
 F 3 "" H 1850 3250 60  0000 C CNN
@@
 P 1500 3250
 F 0 "R2" H 1500 3300 40  0000 C CNN
-F 1 "2.2k" H 1500 3200 40  0000 C CNN
+F 1 "0/2.2k" H 1500 3200 40  0000 C CNN
 F 2 "" H 1500 3250 60  0000 C CNN
 F 3 "" H 1500 3250 60  0000 C CNN
